File: kicad_schematic/wave_flume_daq.kicad_sch (KiCad schematic)
At the start: 39 parts, among them J1 M12 B-5, J2 M12 B-5, J3 M12 B-5, J4 M12 B-5, J5 M12 A-5, J6 M12 A-5, J7 M12 A-5, J8 M12 A-5, J9 C14 inlet, U1 IAA100 (at flume), U2 IAA100 (at flume), U3 IAA100 (at flume)

Commit message: update wire colors and documentation for real install
Connections:
- net AGND: now also J5.4 (4=PWR_GND), J5.4B, J6.4 (4=PWR_GND), J6.4B, J7.4 (4=PWR_GND), J7.4B, J8.3 (3=-OUT), J8.3B, TB10.4, TB10.4B, TB11.4, TB11.4B, TB12.4, TB12.4B, TB13.3, TB13.3B; no longer J5.2 (2=PWR_GND), J5.2B, J6.2 (2=PWR_GND), J6.2B, J7.2 (2=PWR_GND), J7.2B, J8.4 (4=-OUT), J8.4B, TB10.2, TB10.2B, TB11.2, TB11.2B, TB12.2, TB12.2B, TB13.4, TB13.4B
- net GND_12: now also J1.4 (4=PWR_LO), J1.4B, J2.4 (4=PWR_LO), J2.4B, J3.4 (4=PWR_LO), J3.4B, J4.4 (4=PWR_LO), J4.4B, TB6.4, TB6.4B, TB7.4, TB7.4B, TB8.4, TB8.4B, TB9.4, TB9.4B; no longer J1.2 (2=PWR_LO), J1.2B, J2.2 (2=PWR_LO), J2.2B, J3.2 (2=PWR_LO), J3.2B, J4.2 (2=PWR_LO), J4.2B, TB6.2, TB6.2B, TB7.2, TB7.2B, TB8.2, TB8.2B, TB9.2, TB9.2B
- net GND_24ISO: now also J8.4 (4=-EXC), J8.4B, TB13.4, TB13.4B; no longer J8.2 (2=-EXC), J8.2B, TB13.2, TB13.2B
- net WG1_H: now also J1.2 (2=SIG_HI), J1.2B, TB6.2, TB6.2B; no longer J1.3 (3=SIG_HI), J1.3B, TB6.3, TB6.3B
- net WG1_L: now also J1.3 (3=SIG_LO), J1.3B, TB6.3, TB6.3B; no longer J1.4 (4=SIG_LO), J1.4B, TB6.4, TB6.4B
- net WG2_H: now also J2.2 (2=SIG_HI), J2.2B, TB7.2, TB7.2B; no longer J2.3 (3=SIG_HI), J2.3B, TB7.3, TB7.3B
- net WG2_L: now also J2.3 (3=SIG_LO), J2.3B, TB7.3, TB7.3B; no longer J2.4 (4=SIG_LO), J2.4B, TB7.4, TB7.4B
- net WG3_H: now also J3.2 (2=SIG_HI), J3.2B, TB8.2, TB8.2B; no longer J3.3 (3=SIG_HI), J3.3B, TB8.3, TB8.3B
- net WG3_L: now also J3.3 (3=SIG_LO), J3.3B, TB8.3, TB8.3B; no longer J3.4 (4=SIG_LO), J3.4B, TB8.4, TB8.4B
- net WG4_H: now also J4.2 (2=SIG_HI), J4.2B, TB9.2, TB9.2B; no longer J4.3 (3=SIG_HI), J4.3B, TB9.3, TB9.3B
- net WG4_L: now also J4.3 (3=SIG_LO), J4.3B, TB9.3, TB9.3B; no longer J4.4 (4=SIG_LO), J4.4B, TB9.4, TB9.4B
- net LC1_L: now reaches TB10.3B
- net LC1_L: now also A1.37 (CH4L), J5.3 (3=OUT_GND), J5.3B, TB10.3, U1.P4 (OUT_GND)
- net LC3_L: now reaches TB12.3B
- net LC3_L: now also A1.31 (CH6L), J7.3 (3=OUT_GND), J7.3B, TB12.3, U3.P4 (OUT_GND)
- net LC2_L: now reaches TB11.3B
- net LC2_L: now also A1.34 (CH5L), J6.3 (3=OUT_GND), J6.3B, TB11.3, U2.P4 (OUT_GND)
- net F1_H renamed LC1_SHUNT
- net LC1_SHUNT: now also U1.P3 (SHUNT); no longer A1.38 (CH4H), TB10.5B, U1.P5 (VOUT)
- removed net F1_L: A1.37 (CH4L), J5.4 (4=OUT_GND), J5.4B, TB10.4, TB10.4B, U1.P4 (OUT_GND)
- removed net F1_SHUNT: J5.3 (3=SHUNT), J5.3B, TB10.3, U1.P3 (SHUNT)
- net F2_H renamed LC2_SHUNT
- net LC2_SHUNT: now also U2.P3 (SHUNT); no longer A1.35 (CH5H), TB11.5B, U2.P5 (VOUT)
- removed net F2_L: A1.34 (CH5L), J6.4 (4=OUT_GND), J6.4B, TB11.4, TB11.4B, U2.P4 (OUT_GND)
- removed net F2_SHUNT: J6.3 (3=SHUNT), J6.3B, TB11.3, U2.P3 (SHUNT)
- net F3_H renamed LC3_SHUNT
- net LC3_SHUNT: now also U3.P3 (SHUNT); no longer A1.32 (CH6H), TB12.5B, U3.P5 (VOUT)
- removed net F3_L: A1.31 (CH6L), J7.4 (4=OUT_GND), J7.4B, TB12.4, TB12.4B, U3.P4 (OUT_GND)
- removed net F3_SHUNT: J7.3 (3=SHUNT), J7.3B, TB12.3, U3.P3 (SHUNT)
- removed net PS1_H: A1.29 (CH7H), J8.3 (3=+OUT), J8.3B, PT1.3 (+OUT_(yel/grn)), TB13.3, TB13.3B
- new net LC1_H: A1.38 (CH4H), J5.2 (2=VOUT), J5.2B, TB10.2, TB10.2B, U1.P5 (VOUT)
- new net LC2_H: A1.35 (CH5H), J6.2 (2=VOUT), J6.2B, TB11.2, TB11.2B, U2.P5 (VOUT)
- new net LC3_H: A1.32 (CH6H), J7.2 (2=VOUT), J7.2B, TB12.2, TB12.2B, U3.P5 (VOUT)
- new net PT1_H: A1.29 (CH7H), J8.2 (2=+OUT), J8.2B, PT1.3 (+OUT_(yel/grn)), TB13.2, TB13.2B
Other:
- note added: "1. TB-J1..J4 (gauges): term 2 (SigHi, white) -> CH0H-CH3H = pins 1, 4, 7, 10. Term 3 (SigLo, blue) -> CH0L-CH3L = pins 2, 5, 8, 11."
- note added: "2. TB-J5: term 2 (Vout, yellow) -> pin 38 CH4H, term 3 (OutGnd, green) -> pin 37 CH4L."
- note added: "3. TB-J6: term 2 -> pin 35 CH5H, term 3 -> pin 34 CH5L. TB-J7: term 2 -> pin 32 CH6H, term 3 -> pin 31 CH6L."
- note added: "3x LOAD CELLS - integral 5 ft cable wires directly into the IAA100 sensor block; amps live AT THE FLUME (keep them dry). Amp power + output pass through J5-J7. Cable as built: 1 red +VIN, 2 wht VOUT, 3 blu OUT_GND, 4 blk PWR_GND, 5 org SHUNT."
- note added: "4. TB-J8 (pressure): term 2 (+Out, white) -> pin 29 CH7H, term 3 (-Out, blue) -> pin 28 CH7L. Term 3 ALSO keeps its GND-bus wire (isolation island reference)."
- note added: "4x WAVE HEIGHT GAUGES - runs W1-W4, cable as built: 1 red = PWR_HI, 2 grn = SIG_HI, 3 wht = SIG_LO, 4 blk = PWR_LO, 5 = shield drain (twist SIG_HI with SIG_LO). Gauge bonds PWR_LO to SHIELD internally."
- note added: "EARTH = panel earth stud (mains inlet PE + Setra case/shield). SHUNT leads park on TB-J5..J7 terminal 5 (back side empty); touch to +24V momentarily for shunt cal."
- note added: "G5 = Setra -Out island tie (PT1_L)"
- note added: "J1-J4 'shield' = the drain from gauge pin D: land it on contact 5, NOT on the SH shield shell - the single-point ground lives at the GND bus only."
- note added: "M12 pigtail color code, A- and B-code alike (verify on the TE insert): contact 1 = brown, 2 = white, 3 = blue, 4 = black, 5 = gray. As built: 1 = PWR+, 2 = SIG HI, 3 = SIG LO / analog ref, 4 = PWR-, 5 = shield (WG/PT) or SHUNT (LC). Label each lead before trimming."
- note added: "PT1_L (Setra -Out) also ties to the GND bus - the isolation island's only reference."
- note added: "REFERENCE JUMPER (new for differential): one BLUE wire from A6 (GND_24) to the GND bus. The amps' OutGnd pins are now CH4L-CH6L inputs, so this is the force island's only path to AGND."
- note removed: "1. TB-J1..J4 (gauges): term 3 (SigHi, white) -> CH0H-CH3H = pins 1, 4, 7, 10. Term 4 (SigLo, blue) -> CH0L-CH3L = pins 2, 5, 8, 11."
- note removed: "2. TB-J5: term 5 (Vout, yellow) -> pin 38 CH4H, term 4 (OutGnd, green) -> pin 37 CH4L."
- note removed: "3. TB-J6: term 5 -> pin 35 CH5H, term 4 -> pin 34 CH5L. TB-J7: term 5 -> pin 32 CH6H, term 4 -> pin 31 CH6L."
- note removed: "3x LOAD CELLS - integral 5 ft cable wires directly into the IAA100 sensor block; amps live AT THE FLUME (keep them dry). Amp power + output pass through J5-J7."
- note removed: "4. TB-J8 (pressure): term 3 (+Out, white) -> pin 29 CH7H, term 4 (-Out, blue) -> pin 28 CH7L. Term 4 ALSO keeps its GND-bus wire (isolation island reference)."
- note removed: "4x WAVE HEIGHT GAUGES - runs W1-W4 = twisted bundles of 5 single 20 AWG wires (twist SIG_HI wht with SIG_LO blk). Gauge bonds PWR_LO to SHIELD internally."
- note removed: "EARTH = panel earth stud (mains inlet PE + Setra case/shield). SHUNT leads park on TB-J5..J7 terminal 3 (back side empty); touch to +24V momentarily for shunt cal."
- note removed: "G5 = Setra -Out island tie (PS1_L)"
- note removed: "J1-J4 'shield' = a black wire from gauge pin D: land it on contact 5, NOT on the SH shield shell - the single-point ground lives at the GND bus only."
- note removed: "M12 pigtail color code, A- and B-code alike (verify on the TE insert): contact 1 = brown, 2 = white, 3 = blue, 4 = black, 5 = gray. Label each lead before trimming."
- note removed: "PS1_L (Setra -Out) also ties to the GND bus - the isolation island's only reference."
- note removed: "REFERENCE JUMPER (new for differential): one BLUE wire from A6 (GND_24) to the GND bus. The amps' OutGnd pins are now CH0L-CH2L inputs, so this is the force island's only path to AGND."

Commit message: clean up text in docs
Other:
- note added: "J1-J4 = M12 B-code 5-pos: TE T4110402051-000 screw-terminal plug on the cable (heat-shrink at the gland); TE T4171010405-002 receptacle -> DIN rails."
- note added: "J5-J8 = M12 A-code 5-pos: field wires -> TE T4110001051-000 screw-terminal plug; panel side TE T4171010005-002 male receptacle, 0.5 m pigtail -> DIN rails."
- note removed: "J1-J4 = M12 B-code 5-pos: Phoenix SACC-M12FSB-5PL SH (1424664) push-lock plug on the wire bundle (heat-shrink at the gland); TE T4171010405-002 receptacle -> DIN rails."
- note removed: "J5-J8 = M12 A-code 5-pos: field wires -> Phoenix SACC-M12FS-5PL (1424652) push-lock plug; panel side TE T4171010005-002 male receptacle, 0.5 m pigtail -> DIN rails."
Changed lines of the file:
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@@
 		)
 	)
-	(text "J5-J8 = M12 A-code 5-pos: field wires -> Phoenix SACC-M12FS-5PL (1424652) push-lock plug; panel side TE T4171010005-002 male receptacle, 0.5 m pigtail -> DIN rails."
+	(text "J5-J8 = M12 A-code 5-pos: field wires -> TE T4110001051-000 screw-terminal plug; panel side TE T4171010005-002 male receptacle, 0.5 m pigtail -> DIN rails."
 		(exclude_from_sim no)
 		(at 30.48 146.05 0)
@@
 		)
 	)
-	(text "J1-J4 = M12 B-code 5-pos: Phoenix SACC-M12FSB-5PL SH (1424664) push-lock plug on the wire bundle (heat-shrink at the gland); TE T4171010405-002 receptacle -> DIN rails."
+	(text "J1-J4 = M12 B-code 5-pos: TE T4110402051-000 screw-terminal plug on the cable (heat-shrink at the gland); TE T4171010405-002 receptacle -> DIN rails."
 		(exclude_from_sim no)
 		(at 30.48 36.83 0)
